Commit message: URDF: sensors re-measured after the battery went in under the Jetson (2026-09-24)
Lidar 0.16 m forward of the rear axle, scan plane 0.27 m above the floor;
camera lens 0.32 m forward, 0.215 m above the floor, about 5 deg down by tape
and eye - the pitch, roll and height are provisional until the floor plane fit
replaces them. The IMU is on the frame and did not move.

File: jetnano_description/urdf/jetnano.urdf.xacro (robot description, xacro)
@@ -39,25 +39,29 @@
   <xacro:property name="steer_limit"      value="0.5236"/> <!-- 30 degrees -->
   <!-- Where the sensors are bolted, relative to base_link (the middle of
-       the wheelbase, on the axle line). Tape-measured 2026-09-22: the lidar
-       is 0.15 m and the camera 0.29 m forward of the rear axle, so -0.015 m
-       and +0.125 m from base_link; the lidar's scan plane is 0.225 m above
-       the floor, 0.160 above the axle line. The IMU's position is still an
-       estimate. The ORIENTATIONS were checked on the robot
-       2026-09-22: lidar 0 deg is the nose and angles run
-       counter-clockwise (REP-103), the camera image is upright, and the
-       BNO055 is bolted upside down, turned 90 deg and tilted 10 deg on its
-       bracket - the sensor's +y is the robot's +x, its +x the robot's +y,
-       its +z the robot's -z. imu_rpy is the rotation from the tilt routine
-       (docs/bench-calibration-2026-09-21.md), exact to a couple of degrees.
-       The tilt guard reads it back through TF, so this is the only place
-       it lives. -->
-  <xacro:property name="lidar_xyz"  value="-0.015 0.0 0.160"/>
+       the wheelbase, on the axle line, 0.165 m forward of the rear axle and
+       wheel_radius above the floor). Tape-measured 2026-09-24, after the
+       battery went in under the Jetson and raised the whole stack: the lidar
+       is 0.16 m and the camera 0.32 m forward of the rear axle, so -0.005 m
+       and +0.155 m from base_link; the lidar's scan plane is 0.27 m above
+       the floor (0.205 above the axle line - it now looks OVER anything
+       lower than that; the camera covers the gap). The IMU is on the frame
+       and did not move; its position is still an estimate. The ORIENTATIONS
+       were checked on the robot 2026-09-22: lidar 0 deg is the nose and
+       angles run counter-clockwise (REP-103), the camera image is upright,
+       and the BNO055 is bolted upside down, turned 90 deg and tilted 10 deg
+       on its bracket - the sensor's +y is the robot's +x, its +x the robot's
+       +y, its +z the robot's -z. imu_rpy is the rotation from the tilt
+       routine (docs/bench-calibration-2026-09-21.md), exact to a couple of
+       degrees. The tilt guard reads it back through TF, so this is the only
+       place it lives. -->
+  <xacro:property name="lidar_xyz"  value="-0.005 0.0 0.205"/>
   <xacro:property name="lidar_rpy"  value="0 0 0"/>
-  <!-- Camera re-mounted 2026-09-22 below the lidar plane and pitched down:
-       27.1 deg down, +0.9 deg roll, lens 0.178 m above the floor, all from a
-       plane fit to the floor in the aligned depth (0.1 mm residual).
-       z = 0.178 - wheel_radius. -->
-  <xacro:property name="camera_xyz" value="0.125 0.0 0.113"/>
-  <xacro:property name="camera_rpy" value="0.016 0.473 0"/>
+  <!-- Camera re-mounted 2026-09-24: lens 0.215 m above the floor (z = 0.215
+       - wheel_radius), about 5 deg down by eye. PROVISIONAL: the pitch, roll
+       and height are to be replaced by a plane fit to the floor in the depth
+       image, as on 2026-09-22 (27.1 deg down then, 0.1 mm residual) - nvblox
+       puts the floor in the map as an obstacle if this is a few degrees off. -->
+  <xacro:property name="camera_xyz" value="0.155 0.0 0.150"/>
+  <xacro:property name="camera_rpy" value="0 0.087 0"/>
   <xacro:property name="imu_xyz"    value="0.0 0.0 0.060"/>
   <xacro:property name="imu_rpy"    value="2.9698 0.0552 1.5680"/>

Commit message: URDF: camera attitude from the floor plane fit after the 2026-09-24 remount
10.5 deg down, 5.6 deg roll, lens 0.191 m above the floor (39 000 points,
3 mm residual) in place of the tape-and-eye guess; calibration doc updated.

File: jetnano_description/urdf/jetnano.urdf.xacro (robot description, xacro)
@@ -57,11 +57,13 @@
   <xacro:property name="lidar_xyz"  value="-0.005 0.0 0.205"/>
   <xacro:property name="lidar_rpy"  value="0 0 0"/>
-  <!-- Camera re-mounted 2026-09-24: lens 0.215 m above the floor (z = 0.215
-       - wheel_radius), about 5 deg down by eye. PROVISIONAL: the pitch, roll
-       and height are to be replaced by a plane fit to the floor in the depth
-       image, as on 2026-09-22 (27.1 deg down then, 0.1 mm residual) - nvblox
-       puts the floor in the map as an obstacle if this is a few degrees off. -->
-  <xacro:property name="camera_xyz" value="0.155 0.0 0.150"/>
-  <xacro:property name="camera_rpy" value="0 0.087 0"/>
+  <!-- Camera re-mounted 2026-09-24 ("about 5 deg down" by eye): measured on
+       the floor with ros2_gpu_robot tools/camera_pitch.py, a plane fit to the
+       floor in the depth image - 10.5 deg down, 5.6 deg roll (left side up),
+       lens 0.191 m above the floor, 39 000 points, 3 mm mean residual.
+       z = 0.191 - wheel_radius. Re-run the tool whenever the mount moves:
+       nvblox puts the floor in the map as an obstacle if this is a few
+       degrees off. -->
+  <xacro:property name="camera_xyz" value="0.155 0.0 0.126"/>
+  <xacro:property name="camera_rpy" value="0.098 0.183 0"/>
   <xacro:property name="imu_xyz"    value="0.0 0.0 0.060"/>
   <xacro:property name="imu_rpy"    value="2.9698 0.0552 1.5680"/>

Commit message: URDF: the lidar is mounted backwards since the remount - yaw 180 deg
Heading by heading its ranges matched the camera's only once turned 180 deg
(0.2 m median difference; a 1 deg sweep preferred 176-179). Calibration doc.

File: jetnano_description/urdf/jetnano.urdf.xacro (robot description, xacro)
@@ -56,5 +56,12 @@
        place it lives. -->
   <xacro:property name="lidar_xyz"  value="-0.005 0.0 0.205"/>
-  <xacro:property name="lidar_rpy"  value="0 0 0"/>
+  <!-- Mounted BACKWARDS since the 2026-09-24 remount: the lidar's 0 deg is
+       the robot's tail. Found on the floor - the lidar drew the wall behind
+       the robot in front of it, 2.5 m from where the camera put the real
+       one; rotated 180 deg its profile matches the camera's to 0.2 m
+       (a 1 deg sweep prefers 176-179, which is 180 within the method).
+       Fixing it here instead of unbolting it; if the lidar is ever turned
+       round again, this goes back to 0. -->
+  <xacro:property name="lidar_rpy"  value="0 0 ${pi}"/>
   <!-- Camera re-mounted 2026-09-24 ("about 5 deg down" by eye): measured on
        the floor with ros2_gpu_robot tools/camera_pitch.py, a plane fit to the

Commit message: Measured outline (tyre to tyre 0.444 x 0.295 m): Nav2 footprint was 7.5 cm too narrow; lidar scan plane 0.263 m

File: jetnano_description/urdf/jetnano.urdf.xacro (robot description, xacro)
@@ -55,5 +55,8 @@
        degrees. The tilt guard reads it back through TF, so this is the only
        place it lives. -->
-  <xacro:property name="lidar_xyz"  value="-0.005 0.0 0.205"/>
+  <!-- 2026-09-27, Steve's tape: the spinning head spans 0.255-0.271 m above the
+       floor, so the scan plane (mid-head) is ~0.263 m: z = 0.263 - 0.065 = 0.198.
+       Overall, tyre to tyre: 0.444 m long, 0.295 m wide, 0.27 m tall (lidar top). -->
+  <xacro:property name="lidar_xyz"  value="-0.005 0.0 0.198"/>
   <!-- Mounted BACKWARDS since the 2026-09-24 remount: the lidar's 0 deg is
        the robot's tail. Found on the floor - the lidar drew the wall behind

Commit message: Camera mounted upside down (USB extension gone): URDF roll 180, re-measured pitch; pages turn the picture
- jetnano.urdf.xacro camera_rpy 3.130 -0.118 0, z 0.048: plane fit on the floor
  right after the flip - 6.8 deg up, roll 179.3, lens 0.113 m, 34 166 inliers,
  3 mm mean residual. cuVSLAM and nvblox follow through TF.
- csi_cameras: d435_rotate parameter (robot.launch.py: 180) served as
  /config.json; index.html and dash.html rotate the RealSense picture with CSS,
  so it costs the robot nothing.

File: jetnano_description/urdf/jetnano.urdf.xacro (robot description, xacro)
@@ -48,5 +48,6 @@
        and did not move; its position is still an estimate. The ORIENTATIONS
        were checked on the robot 2026-09-22: lidar 0 deg is the nose and
-       angles run counter-clockwise (REP-103), the camera image is upright,
+       angles run counter-clockwise (REP-103), the camera image is upright
+       (until 2026-09-27; the camera is now upside down, see camera_rpy),
        and the BNO055 is bolted upside down, turned 90 deg and tilted 10 deg
        on its bracket - the sensor's +y is the robot's +x, its +x the robot's
@@ -78,7 +79,14 @@
        held by tape for now. Plane fit the same evening: 7.8 deg UP (pitch
        -0.136), 1.2 deg roll, lens 0.112 m above the floor (Steve measured 0.11),
-       31 837 inlier points, 3 mm mean residual. -->
-  <xacro:property name="camera_xyz" value="0.185 0.0 0.047"/>
-  <xacro:property name="camera_rpy" value="-0.021 -0.136 0"/>
+       31 837 inlier points, 3 mm mean residual.
+       Turned UPSIDE DOWN 2026-09-27 (Steve: its USB port now faces the Jetson's,
+       and the USB extension is gone - the suspect in the camera dropouts). Roll
+       ~180 deg says so; cuVSLAM and nvblox take it from here through TF, and the
+       web pages turn the picture back (csi_cameras d435_rotate). Plane fit right
+       after (camera_pitch.py with its upside-down option): 6.8 deg UP (pitch -0.118), roll
+       179.3 deg, lens 0.113 m above the floor, 34 166 inliers, 3 mm mean residual.
+       If it is ever turned back upright: roll back to ~0 and d435_rotate 0. -->
+  <xacro:property name="camera_xyz" value="0.185 0.0 0.048"/>
+  <xacro:property name="camera_rpy" value="3.130 -0.118 0"/>
   <xacro:property name="imu_xyz"    value="0.0 0.0 0.060"/>
   <xacro:property name="imu_rpy"    value="2.9698 0.0552 1.5680"/>
