Commit message: Put the measured IMU mount in the URDF and rotate the tilt guard into base_link
The BNO055 is bolted upside down, turned 90 degrees and tilted 10 degrees,
measured 2026-09-22 by tipping the robot by hand: the driver reports a
parked robot as rolled 170 degrees. imu_rpy now carries that rotation, and
the tilt guard looks it up from TF (or takes imu_mount_rpy) and rotates
every sample into base_link before judging it, with tests against the
real rest reading. Lidar and camera orientations were verified as-is.

Co-Authored-By: Claude Fable 5.1 <noreply@anthropic.com>
Claude-Session: https://claude.ai/code/session_018b3JVpbw8hhHjzcEWK6tKC

File: jetnano_description/urdf/jetnano.urdf.xacro (robot description, xacro)
@@ -37,5 +37,14 @@
   <xacro:property name="chassis_z_offset" value="0.010"/>  <!-- chassis centre above axle line -->
   <xacro:property name="steer_limit"      value="0.5236"/> <!-- 30 degrees -->
-  <!-- MEASURE ME - where the sensors are bolted, relative to base_link -->
+  <!-- Where the sensors are bolted, relative to base_link. Positions are
+       still estimates (tape measure pending); the ORIENTATIONS were checked
+       on the robot 2026-09-22: lidar 0 deg is the nose and angles run
+       counter-clockwise (REP-103), the camera image is upright, and the
+       BNO055 is bolted upside down, turned 90 deg and tilted 10 deg on its
+       bracket - the sensor's +y is the robot's +x, its +x the robot's +y,
+       its +z the robot's -z. imu_rpy is the rotation from the tilt routine
+       (docs/bench-calibration-2026-09-21.md), exact to a couple of degrees.
+       The tilt guard reads it back through TF, so this is the only place
+       it lives. -->
   <xacro:property name="lidar_xyz"  value="0.0 0.0 0.145"/>
   <xacro:property name="lidar_rpy"  value="0 0 0"/>
@@ -43,5 +52,5 @@
   <xacro:property name="camera_rpy" value="0 0 0"/>
   <xacro:property name="imu_xyz"    value="0.0 0.0 0.060"/>
-  <xacro:property name="imu_rpy"    value="0 0 0"/>
+  <xacro:property name="imu_rpy"    value="2.9698 0.0552 1.5680"/>
   <!-- Rough masses. Good enough for TF and RViz; revisit only if you ever
        simulate the robot dynamically. -->

Commit message: URDF: the camera's measured pitch, roll and height
Plane fit to the floor in the aligned depth with the robot on the ground:
27.1 deg down, +0.9 deg roll, lens 0.178 m up. Three identical readings,
0.1 mm residual, cross-checked against the depth at the image centre.

Co-Authored-By: Claude Fable 5.1 <noreply@anthropic.com>
Claude-Session: https://claude.ai/code/session_018b3JVpbw8hhHjzcEWK6tKC

File: jetnano_description/urdf/jetnano.urdf.xacro (robot description, xacro)
@@ -49,6 +49,10 @@
   <xacro:property name="lidar_xyz"  value="0.0 0.0 0.145"/>
   <xacro:property name="lidar_rpy"  value="0 0 0"/>
-  <xacro:property name="camera_xyz" value="0.150 0.0 0.095"/>
-  <xacro:property name="camera_rpy" value="0 0 0"/>
+  <!-- Camera re-mounted 2026-09-22 below the lidar plane and pitched down:
+       27.1 deg down, +0.9 deg roll, lens 0.178 m above the floor, all from a
+       plane fit to the floor in the aligned depth (0.1 mm residual). x is
+       still a tape-measure job; z = 0.178 - wheel_radius. -->
+  <xacro:property name="camera_xyz" value="0.150 0.0 0.118"/>
+  <xacro:property name="camera_rpy" value="0.016 0.473 0"/>
   <xacro:property name="imu_xyz"    value="0.0 0.0 0.060"/>
   <xacro:property name="imu_rpy"    value="2.9698 0.0552 1.5680"/>

Commit message: Tape-measured chassis geometry: 0.330 wheelbase, 0.230 track, 0.065 wheels
Plus the lidar and camera positions along the chassis (0.15 and 0.29 m
forward of the rear axle). Sim steering geometry, its tests, the Nav2
turning-radius note and the tilt guard's rationale follow the same numbers.

Co-Authored-By: Claude Fable 5.1 <noreply@anthropic.com>
Claude-Session: https://claude.ai/code/session_018b3JVpbw8hhHjzcEWK6tKC

File: jetnano_description/urdf/jetnano.urdf.xacro (robot description, xacro)
@@ -26,9 +26,10 @@
 <robot name="jetnano" xmlns:xacro="http://www.ros.org/wiki/xacro">
   <!-- ============================================================
-       MEASURE ME - chassis geometry (metres, radians)
-       ============================================================ -->
-  <xacro:property name="wheelbase"        value="0.313"/>  <!-- front axle to rear axle -->
-  <xacro:property name="track_width"      value="0.220"/>  <!-- left wheel to right wheel -->
-  <xacro:property name="wheel_radius"     value="0.060"/>  <!-- tyre radius, loaded -->
+       Chassis geometry (metres, radians). Wheelbase, track and tyre
+       radius tape-measured 2026-09-22; the body box is still an estimate.
+       ============================================================ -->
+  <xacro:property name="wheelbase"        value="0.330"/>  <!-- front axle to rear axle -->
+  <xacro:property name="track_width"      value="0.230"/>  <!-- left wheel to right wheel -->
+  <xacro:property name="wheel_radius"     value="0.065"/>  <!-- tyre radius, loaded -->
   <xacro:property name="wheel_width"      value="0.045"/>
   <xacro:property name="chassis_length"   value="0.400"/>
@@ -37,7 +38,10 @@
   <xacro:property name="chassis_z_offset" value="0.010"/>  <!-- chassis centre above axle line -->
   <xacro:property name="steer_limit"      value="0.5236"/> <!-- 30 degrees -->
-  <!-- Where the sensors are bolted, relative to base_link. Positions are
-       still estimates (tape measure pending); the ORIENTATIONS were checked
-       on the robot 2026-09-22: lidar 0 deg is the nose and angles run
+  <!-- Where the sensors are bolted, relative to base_link (the middle of
+       the wheelbase, on the axle line). Tape-measured 2026-09-22: the lidar
+       is 0.15 m and the camera 0.29 m forward of the rear axle, so -0.015 m
+       and +0.125 m from base_link. The lidar's height and the IMU's position
+       are still estimates. The ORIENTATIONS were checked on the robot
+       2026-09-22: lidar 0 deg is the nose and angles run
        counter-clockwise (REP-103), the camera image is upright, and the
        BNO055 is bolted upside down, turned 90 deg and tilted 10 deg on its
@@ -47,11 +51,11 @@
        The tilt guard reads it back through TF, so this is the only place
        it lives. -->
-  <xacro:property name="lidar_xyz"  value="0.0 0.0 0.145"/>
+  <xacro:property name="lidar_xyz"  value="-0.015 0.0 0.145"/>
   <xacro:property name="lidar_rpy"  value="0 0 0"/>
   <!-- Camera re-mounted 2026-09-22 below the lidar plane and pitched down:
        27.1 deg down, +0.9 deg roll, lens 0.178 m above the floor, all from a
-       plane fit to the floor in the aligned depth (0.1 mm residual). x is
-       still a tape-measure job; z = 0.178 - wheel_radius. -->
-  <xacro:property name="camera_xyz" value="0.150 0.0 0.118"/>
+       plane fit to the floor in the aligned depth (0.1 mm residual).
+       z = 0.178 - wheel_radius. -->
+  <xacro:property name="camera_xyz" value="0.125 0.0 0.113"/>
   <xacro:property name="camera_rpy" value="0.016 0.473 0"/>
   <xacro:property name="imu_xyz"    value="0.0 0.0 0.060"/>

Commit message: URDF: measured lidar height (0.225 m above the floor)
Co-Authored-By: Claude Fable 5.1 <noreply@anthropic.com>
Claude-Session: https://claude.ai/code/session_018b3JVpbw8hhHjzcEWK6tKC

File: jetnano_description/urdf/jetnano.urdf.xacro (robot description, xacro)
@@ -41,6 +41,7 @@
        the wheelbase, on the axle line). Tape-measured 2026-09-22: the lidar
        is 0.15 m and the camera 0.29 m forward of the rear axle, so -0.015 m
-       and +0.125 m from base_link. The lidar's height and the IMU's position
-       are still estimates. The ORIENTATIONS were checked on the robot
+       and +0.125 m from base_link; the lidar's scan plane is 0.225 m above
+       the floor, 0.160 above the axle line. The IMU's position is still an
+       estimate. The ORIENTATIONS were checked on the robot
        2026-09-22: lidar 0 deg is the nose and angles run
        counter-clockwise (REP-103), the camera image is upright, and the
@@ -51,5 +52,5 @@
        The tilt guard reads it back through TF, so this is the only place
        it lives. -->
-  <xacro:property name="lidar_xyz"  value="-0.015 0.0 0.145"/>
+  <xacro:property name="lidar_xyz"  value="-0.015 0.0 0.160"/>
   <xacro:property name="lidar_rpy"  value="0 0 0"/>
   <!-- Camera re-mounted 2026-09-22 below the lidar plane and pitched down:

Commit message: urdf: the D435 moved low between the front wheels (0.35 m ahead of the rear axle, 0.11 m up); tilt provisional until the plane fit
Co-Authored-By: Claude Opus 5.5 <noreply@anthropic.com>

File: jetnano_description/urdf/jetnano.urdf.xacro (robot description, xacro)
@@ -70,7 +70,11 @@
        z = 0.191 - wheel_radius. Re-run the tool whenever the mount moves:
        nvblox puts the floor in the map as an obstacle if this is a few
-       degrees off. -->
-  <xacro:property name="camera_xyz" value="0.155 0.0 0.126"/>
-  <xacro:property name="camera_rpy" value="0.098 0.183 0"/>
+       degrees off.
+       Moved again 2026-09-25 (Steve, to make room for the pan-tilt camera): low
+       between the front wheels, 0.35 m ahead of the rear axle (x = 0.35 - 0.165),
+       its centre 0.11 m off the floor (z = 0.11 - wheel_radius), held by tape for
+       now. The tilt below is PROVISIONAL (level) until the plane fit is re-run. -->
+  <xacro:property name="camera_xyz" value="0.185 0.0 0.045"/>
+  <xacro:property name="camera_rpy" value="0 0 0"/>
   <xacro:property name="imu_xyz"    value="0.0 0.0 0.060"/>
   <xacro:property name="imu_rpy"    value="2.9698 0.0552 1.5680"/>

Commit message: urdf: the low D435 measured by plane fit - 7.8 deg up, 1.2 deg roll, lens 0.112 m
Co-Authored-By: Claude Opus 5.5 <noreply@anthropic.com>

File: jetnano_description/urdf/jetnano.urdf.xacro (robot description, xacro)
@@ -73,8 +73,9 @@
        Moved again 2026-09-25 (Steve, to make room for the pan-tilt camera): low
        between the front wheels, 0.35 m ahead of the rear axle (x = 0.35 - 0.165),
-       its centre 0.11 m off the floor (z = 0.11 - wheel_radius), held by tape for
-       now. The tilt below is PROVISIONAL (level) until the plane fit is re-run. -->
-  <xacro:property name="camera_xyz" value="0.185 0.0 0.045"/>
-  <xacro:property name="camera_rpy" value="0 0 0"/>
+       held by tape for now. Plane fit the same evening: 7.8 deg UP (pitch
+       -0.136), 1.2 deg roll, lens 0.112 m above the floor (Steve measured 0.11),
+       31 837 inlier points, 3 mm mean residual. -->
+  <xacro:property name="camera_xyz" value="0.185 0.0 0.047"/>
+  <xacro:property name="camera_rpy" value="-0.021 -0.136 0"/>
   <xacro:property name="imu_xyz"    value="0.0 0.0 0.060"/>
   <xacro:property name="imu_rpy"    value="2.9698 0.0552 1.5680"/>

Commit message: Camera re-seated (roll 183.2, pitch 4.9 up, lens 0.109 m); stop pictures right side up
Steve re-seated the D435 (pushed left and crooked). Floor plane fit: 27 012 inliers,
3.6 mm residual. nav_helper turns the RealSense stop picture as the pages do.

Co-Authored-By: Claude Opus 5.5 <noreply@anthropic.com>
Claude-Session: https://claude.ai/code/session_014rgB5QvcLgVwPqyJKQKtcY

File: jetnano_description/urdf/jetnano.urdf.xacro (robot description, xacro)
@@ -86,7 +86,12 @@
        after (camera_pitch.py with its upside-down option): 6.8 deg UP (pitch -0.118), roll
        179.3 deg, lens 0.113 m above the floor, 34 166 inliers, 3 mm mean residual.
-       If it is ever turned back upright: roll back to ~0 and d435_rotate 0. -->
-  <xacro:property name="camera_xyz" value="0.185 0.0 0.048"/>
-  <xacro:property name="camera_rpy" value="3.130 -0.118 0"/>
+       If it is ever turned back upright: roll back to ~0 and d435_rotate 0.
+       Re-seated 2026-10-09 (Steve: it was pushed left and crooked). Plane fit on the great-room
+       floor: 4.9 deg UP (pitch -0.085), roll 183.2 deg (-3.086), lens 0.109 m above the floor,
+       27 012 inliers, 3.6 mm mean residual. The High Accuracy preset (since 10-02) drops the
+       near floor, so the fit needs depth_module.visual_preset 1 for a minute - and changing it
+       live restarts the camera driver (the watchdog brings it back). -->
+  <xacro:property name="camera_xyz" value="0.185 0.0 0.044"/>
+  <xacro:property name="camera_rpy" value="-3.086 -0.085 0"/>
   <xacro:property name="imu_xyz"    value="0.0 0.0 0.060"/>
   <xacro:property name="imu_rpy"    value="2.9698 0.0552 1.5680"/>

Commit message: Camera aim: 7 deg left (depth vs lidar on walls, two spots)
Co-Authored-By: Claude Opus 5.5 <noreply@anthropic.com>
Claude-Session: https://claude.ai/code/session_014rgB5QvcLgVwPqyJKQKtcY

File: jetnano_description/urdf/jetnano.urdf.xacro (robot description, xacro)
@@ -91,7 +91,11 @@
        27 012 inliers, 3.6 mm mean residual. The High Accuracy preset (since 10-02) drops the
        near floor, so the fit needs depth_module.visual_preset 1 for a minute - and changing it
-       live restarts the camera driver (the watchdog brings it back). -->
+       live restarts the camera driver (the watchdog brings it back).
+       Aim (yaw) the same day, its depth matched against the lidar on the walls 0.16-0.26 m up,
+       turning about the lens: 8.5 and 6.0 deg LEFT at two spots / headings (5 at a third, before
+       the plane fit) -> 7 deg (0.122). A sideways offset is not measurable that way (it trades
+       against the turn along the walls), so y stays 0. -->
   <xacro:property name="camera_xyz" value="0.185 0.0 0.044"/>
-  <xacro:property name="camera_rpy" value="-3.086 -0.085 0"/>
+  <xacro:property name="camera_rpy" value="-3.086 -0.085 0.122"/>
   <xacro:property name="imu_xyz"    value="0.0 0.0 0.060"/>
   <xacro:property name="imu_rpy"    value="2.9698 0.0552 1.5680"/>
